File: spdif-pmod.sch (KiCad schematic (older format))
At the start: 9 parts, among them J1 PMOD, J2 COAX_OUT, U1 74LVC1G34, U2 OPTICAL_OUT

Commit message: Correct Murata part that would be used instead
Other:
- note added: "The official spec apparently calls for a pulse transformer on the coax output.\nThis should be good enough for most cases though.\nThe Murata DA101(J)C could be used if one is needed."
- note removed: "The official spec apparently calls for a pulse transformer on the coax output.\nThis should be good enough for most cases though.\nThe Murata DA103C could be used if one is needed."
Changed lines of the file:
@@
 v1.0.3
 Text Notes 3000 3500 0    50   ~ 0
-The official spec apparently calls for a pulse transformer on the coax output.\nThis should be good enough for most cases though.\nThe Murata DA103C could be used if one is needed.
+The official spec apparently calls for a pulse transformer on the coax output.\nThis should be good enough for most cases though.\nThe Murata DA101(J)C could be used if one is needed.
 Text Notes 2600 4150 0    50   ~ 0
 By Dan Rodrigues\n\ngithub.com/dan-rodrigues
